File: Hardware/Fc/Fc.kicad_sch (KiCad schematic)
At the start: 60 parts, among them U1 STM32F407VGTx

Commit message: Added USB
Parts:
- removed C10, C11, C12, C13, C14, C9: 100n, Capacitor_SMD:C_0402_1005Metric, symbol Device:C
- removed D1: STAT, LED_SMD:LED_0402_1005Metric, symbol Device:LED_BGRK
- removed D2: BAT, LED_SMD:LED_0402_1005Metric, symbol Device:LED_BGRK
- removed FATAL1, PWR1, WD1, WD2: R, LED_SMD:LED_0402_1005Metric, symbol Device:LED
- removed GOAL1, NAV1: G, LED_SMD:LED_0402_1005Metric, symbol Device:LED
- removed R10, R13, R18, R19: 2k2, Resistor_SMD:R_0402_1005Metric, symbol Device:R
- removed R11, R12, R14, R15, R16, R17, R20, R9: 1k, Resistor_SMD:R_0402_1005Metric, symbol Device:R
- added C9: 1u, Capacitor_SMD:C_0402_1005Metric, symbol Device:C_Polarized
- added TP4: GND, symbol Connector:TestPoint
- FB1: value FerriteBead_Small -> 120R
Connections:
- net +3V3: now also C9.1
- net GND: now also C9.2, TP4.1
- net LED8: now also U1.7 (PC13); no longer U1.38 (PE7)
- net TIM1_CH4: no longer names the net of U1.45 (PE14)
- net USB_OTG_FS_DM renamed USB_D-
- net USB_OTG_FS_DP renamed USB_D+
- net USB_OTG_FS_ID: no longer names the net of U1.69 (PA10)
- net USB_OTG_FS_VBUS: no longer names the net of U1.68 (PA9)
- net VDDA renamed +3.3VA
- no-connect marks 32 -> 35
Other:
- added sheet Status (Status.kicad_sch)
- note removed: "LED Array"
- moved on the sheet: 25MHz1, BOOT1, C1, C17, C18, C19, C2, C20, C21, C22, C23, C3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

Commit message: Building with new libcamera updates
Parts:
- TP1, TP2, TP3, TP4: footprint (none) -> TestPoint:TestPoint_Pad_2.0x2.0mm
