File: Hardware/Fc/FcPeripherals.kicad_sch (KiCad schematic)
At the start: 36 parts, among them J2 Raspberry_Pi_2_3, J3 Conn_01x02_Male, J4 Conn_01x02_Male, J5 Conn_01x02_Male, J6 Conn_01x02_Male, J7 Conn_01x02_Male, U3 ICM-20602, U5 TLV9001IDCK, U6 TLV9001IDCK, U7 TLV9001IDCK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

Commit message: Building with new libcamera updates
Parts:
- C15, C16, C35: footprint (none) -> Capacitor_SMD:C_0402_1005Metric
- J3, J4, J5, J6, J7: footprint (none) -> Connector_PinHeader_2.54mm:PinHeader_1x02_P2.54mm_Vertical
- R1T1, R1T2, R1T3, R1T4, R1T5, R2T1, R2T2, R2T3, R2T4, R2T5, R3T1, R3T2, R3T3, R3T4, R3T5, R4T1, R4T2, R4T3, R4T4, R4T5: footprint (none) -> Resistor_SMD:R_0402_1005Metric
Changed lines of the file:
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@@
       (effects (font (size 1.27 1.27)) (justify left))
     )
-    (property "Footprint" "" (id 2) (at 121.412 25.4 90)
+    (property "Footprint" "Resistor_SMD:R_0402_1005Metric" (id 2) (at 121.412 25.4 90)
       (effects (font (size 1.27 1.27)) hide)
     )
@@
       (effects (font (size 1.27 1.27)) (justify left))
     )
-    (property "Footprint" "" (id 2) (at 113.03 90.17 0)
+    (property "Footprint" "Connector_PinHeader_2.54mm:PinHeader_1x02_P2.54mm_Vertical" (id 2) (at 113.03 90.17 0)
       (effects (font (size 1.27 1.27)) hide)
     )
@@
       (effects (font (size 1.27 1.27)) (justify left))
     )
-    (property "Footprint" "" (id 2) (at 121.412 134.62 90)
+    (property "Footprint" "Resistor_SMD:R_0402_1005Metric" (id 2) (at 121.412 134.62 90)
       (effects (font (size 1.27 1.27)) hide)
     )
@@
     (property "Reference" "R4T5" (id 0) (at 140.97 134.62 90))
     (property "Value" "1k5" (id 1) (at 140.97 137.16 90))
-    (property "Footprint" "" (id 2) (at 140.97 141.478 90)
+    (property "Footprint" "Resistor_SMD:R_0402_1005Metric" (id 2) (at 140.97 141.478 90)
       (effects (font (size 1.27 1.27)) hide)
     )
@@
       (effects (font (size 1.27 1.27)) (justify left))
     )
-    (property "Footprint" "" (id 2) (at 192.532 25.4 90)
+    (property "Footprint" "Resistor_SMD:R_0402_1005Metric" (id 2) (at 192.532 25.4 90)
       (effects (font (size 1.27 1.27)) hide)
     )
@@
       (effects (font (size 1.27 1.27)) (justify left))
     )
-    (property "Footprint" "" (id 2) (at 111.252 109.22 90)
+    (property "Footprint" "Resistor_SMD:R_0402_1005Metric" (id 2) (at 111.252 109.22 90)
       (effects (font (size 1.27 1.27)) hide)
     )
@@
       (effects (font (size 1.27 1.27)) (justify left))
     )
-    (property "Footprint" "" (id 2) (at 36.5252 31.75 0)
+    (property "Footprint" "Capacitor_SMD:C_0402_1005Metric" (id 2) (at 36.5252 31.75 0)
       (effects (font (size 1.27 1.27)) hide)
     )
@@
       (effects (font (size 1.27 1.27)) (justify left))
     )
-    (property "Footprint" "" (id 2) (at 184.15 90.17 0)
+    (property "Footprint" "Connector_PinHeader_2.54mm:PinHeader_1x02_P2.54mm_Vertical" (id 2) (at 184.15 90.17 0)
       (effects (font (size 1.27 1.27)) hide)
     )
@@
       (effects (font (size 1.27 1.27)) (justify left))
     )
-    (property "Footprint" "" (id 2) (at 184.15 35.56 0)
+    (property "Footprint" "Connector_PinHeader_2.54mm:PinHeader_1x02_P2.54mm_Vertical" (id 2) (at 184.15 35.56 0)
       (effects (font (size 1.27 1.27)) hide)
     )
@@
       (effects (font (size 1.27 1.27)) (justify left))
     )
-    (property "Footprint" "" (id 2) (at 192.532 90.17 90)
+    (property "Footprint" "Resistor_SMD:R_0402_1005Metric" (id 2) (at 192.532 90.17 90)
       (effects (font (size 1.27 1.27)) hide)
     )
@@
       (effects (font (size 1.27 1.27)) (justify left))
     )
-    (property "Footprint" "" (id 2) (at 111.252 54.61 90)
+    (property "Footprint" "Resistor_SMD:R_0402_1005Metric" (id 2) (at 111.252 54.61 90)
       (effects (font (size 1.27 1.27)) hide)
     )
@@
       (effects (font (size 1.27 1.27)) (justify left))
     )
-    (property "Footprint" "" (id 2) (at 64.4652 54.61 0)
+    (property "Footprint" "Capacitor_SMD:C_0402_1005Metric" (id 2) (at 64.4652 54.61 0)
       (effects (font (size 1.27 1.27)) hide)
     )
@@
       (effects (font (size 1.27 1.27)) (justify left))
     )
-    (property "Footprint" "" (id 2) (at 121.412 90.17 90)
+    (property "Footprint" "Resistor_SMD:R_0402_1005Metric" (id 2) (at 121.412 90.17 90)
       (effects (font (size 1.27 1.27)) hide)
     )
@@
       (effects (font (size 1.27 1.27)) (justify left))
     )
-    (property "Footprint" "" (id 2) (at 192.532 35.56 90)
+    (property "Footprint" "Resistor_SMD:R_0402_1005Metric" (id 2) (at 192.532 35.56 90)
       (effects (font (size 1.27 1.27)) hide)
     )
@@
       (effects (font (size 1.27 1.27)) (justify left))
     )
-    (property "Footprint" "" (id 2) (at 111.252 163.83 90)
+    (property "Footprint" "Resistor_SMD:R_0402_1005Metric" (id 2) (at 111.252 163.83 90)
       (effects (font (size 1.27 1.27)) hide)
     )
@@
       (effects (font (size 1.27 1.27)) (justify left))
     )
-    (property "Footprint" "" (id 2) (at 113.03 35.56 0)
+    (property "Footprint" "Connector_PinHeader_2.54mm:PinHeader_1x02_P2.54mm_Vertical" (id 2) (at 113.03 35.56 0)
       (effects (font (size 1.27 1.27)) hide)
     )
@@
     (property "Reference" "R4T3" (id 0) (at 140.97 80.01 90))
     (property "Value" "1k5" (id 1) (at 140.97 82.55 90))
-    (property "Footprint" "" (id 2) (at 140.97 86.868 90)
+    (property "Footprint" "Resistor_SMD:R_0402_1005Metric" (id 2) (at 140.97 86.868 90)
       (effects (font (size 1.27 1.27)) hide)
     )
@@
       (effects (font (size 1.27 1.27)) (justify left))
     )
-    (property "Footprint" "" (id 2) (at 26.3652 31.75 0)
+    (property "Footprint" "Capacitor_SMD:C_0402_1005Metric" (id 2) (at 26.3652 31.75 0)
       (effects (font (size 1.27 1.27)) hide)
     )
@@
       (effects (font (size 1.27 1.27)) (justify left))
     )
-    (property "Footprint" "" (id 2) (at 121.412 144.78 90)
+    (property "Footprint" "Resistor_SMD:R_0402_1005Metric" (id 2) (at 121.412 144.78 90)
       (effects (font (size 1.27 1.27)) hide)
     )
@@
     (property "Reference" "R4T4" (id 0) (at 212.09 80.01 90))
     (property "Value" "1k5" (id 1) (at 212.09 82.55 90))
-    (property "Footprint" "" (id 2) (at 212.09 86.868 90)
+    (property "Footprint" "Resistor_SMD:R_0402_1005Metric" (id 2) (at 212.09 86.868 90)
       (effects (font (size 1.27 1.27)) hide)
     )
@@
       (effects (font (size 1.27 1.27)) (justify left))
     )
-    (property "Footprint" "" (id 2) (at 192.532 80.01 90)
+    (property "Footprint" "Resistor_SMD:R_0402_1005Metric" (id 2) (at 192.532 80.01 90)
       (effects (font (size 1.27 1.27)) hide)
     )
@@
       (effects (font (size 1.27 1.27)) (justify left))
     )
-    (property "Footprint" "" (id 2) (at 182.372 109.22 90)
+    (property "Footprint" "Resistor_SMD:R_0402_1005Metric" (id 2) (at 182.372 109.22 90)
       (effects (font (size 1.27 1.27)) hide)
     )
@@
     (property "Reference" "R4T1" (id 0) (at 140.97 25.4 90))
     (property "Value" "1k5" (id 1) (at 140.97 27.94 90))
-    (property "Footprint" "" (id 2) (at 140.97 32.258 90)
+    (property "Footprint" "Resistor_SMD:R_0402_1005Metric" (id 2) (at 140.97 32.258 90)
       (effects (font (size 1.27 1.27)) hide)
     )
@@
       (effects (font (size 1.27 1.27)) (justify left))
     )
-    (property "Footprint" "" (id 2) (at 121.412 80.01 90)
+    (property "Footprint" "Resistor_SMD:R_0402_1005Metric" (id 2) (at 121.412 80.01 90)
       (effects (font (size 1.27 1.27)) hide)
     )
@@
       (effects (font (size 1.27 1.27)) (justify left))
     )
-    (property "Footprint" "" (id 2) (at 113.03 144.78 0)
+    (property "Footprint" "Connector_PinHeader_2.54mm:PinHeader_1x02_P2.54mm_Vertical" (id 2) (at 113.03 144.78 0)
       (effects (font (size 1.27 1.27)) hide)
     )
@@
       (effects (font (size 1.27 1.27)) (justify left))
     )
-    (property "Footprint" "" (id 2) (at 121.412 35.56 90)
+    (property "Footprint" "Resistor_SMD:R_0402_1005Metric" (id 2) (at 121.412 35.56 90)
       (effects (font (size 1.27 1.27)) hide)
     )
@@
     (property "Reference" "R4T2" (id 0) (at 212.09 25.4 90))
     (property "Value" "1k5" (id 1) (at 212.09 27.94 90))
-    (property "Footprint" "" (id 2) (at 212.09 32.258 90)
+    (property "Footprint" "Resistor_SMD:R_0402_1005Metric" (id 2) (at 212.09 32.258 90)
       (effects (font (size 1.27 1.27)) hide)
     )
@@
       (effects (font (size 1.27 1.27)) (justify left))
     )
-    (property "Footprint" "" (id 2) (at 182.372 54.61 90)
-      (effects (font (size 1.27 1.27)) hide)
-    )
+    (property "Footprint" "Resistor_SMD:R_0402_1005Metric" (id 2) (at 182.372 54.61 90)
+      (effects (font (size 1.27 1.27)) hide)
+    )
