File: Hardware/Fc/Status.kicad_sch (KiCad schematic)
At the start: 40 parts, among them U10 DA04-11SURKWA, U4 MCP23017-E_SO

Commit message: Building with new libcamera updates
Parts:
- C10: footprint (none) -> Capacitor_SMD:C_0402_1005Metric
- R10, R11, R12, R13, R14, R15, R16, R17, R18, R19, R20, R29, R30, R31: footprint (none) -> Resistor_SMD:R_0603_1608Metric
- R9: footprint (none) -> Resistor_SMD:R_0402_1005Metric
Changed lines of the file:
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@@
     (property "Reference" "R10" (id 0) (at 52.07 35.56 90))
     (property "Value" "150R" (id 1) (at 52.07 36.83 90))
-    (property "Footprint" "" (id 2) (at 52.07 38.608 90)
+    (property "Footprint" "Resistor_SMD:R_0603_1608Metric" (id 2) (at 52.07 38.608 90)
       (effects (font (size 1.27 1.27)) hide)
     )
@@
     (property "Reference" "R29" (id 0) (at 95.25 45.72 90))
     (property "Value" "150R" (id 1) (at 95.25 46.99 90))
-    (property "Footprint" "" (id 2) (at 95.25 48.768 90)
+    (property "Footprint" "Resistor_SMD:R_0603_1608Metric" (id 2) (at 95.25 48.768 90)
       (effects (font (size 1.27 1.27)) hide)
     )
@@
     (property "Reference" "R16" (id 0) (at 52.07 50.8 90))
     (property "Value" "150R" (id 1) (at 52.07 52.07 90))
-    (property "Footprint" "" (id 2) (at 52.07 53.848 90)
+    (property "Footprint" "Resistor_SMD:R_0603_1608Metric" (id 2) (at 52.07 53.848 90)
       (effects (font (size 1.27 1.27)) hide)
     )
@@
   (symbol (lib_id "power:GND") (at 144.145 56.515 0) (unit 1)
     (in_bom yes) (on_board yes) (fields_autoplaced)
-    (property "Reference" "#PWR072" (id 0) (at 144.145 62.865 0)
+    (property "Reference" "#PWR0128" (id 0) (at 144.145 62.865 0)
       (effects (font (size 1.27 1.27)) hide)
     )
@@
     (property "Reference" "R13" (id 0) (at 52.07 43.18 90))
     (property "Value" "150R" (id 1) (at 52.07 44.45 90))
-    (property "Footprint" "" (id 2) (at 52.07 46.228 90)
+    (property "Footprint" "Resistor_SMD:R_0603_1608Metric" (id 2) (at 52.07 46.228 90)
       (effects (font (size 1.27 1.27)) hide)
     )
@@
       (effects (font (size 1.27 1.27)) (justify left))
     )
-    (property "Footprint" "" (id 2) (at 28.9052 31.75 0)
+    (property "Footprint" "Capacitor_SMD:C_0402_1005Metric" (id 2) (at 28.9052 31.75 0)
       (effects (font (size 1.27 1.27)) hide)
     )
@@
     (property "Reference" "R19" (id 0) (at 95.25 40.64 90))
     (property "Value" "150R" (id 1) (at 95.25 41.91 90))
-    (property "Footprint" "" (id 2) (at 95.25 43.688 90)
+    (property "Footprint" "Resistor_SMD:R_0603_1608Metric" (id 2) (at 95.25 43.688 90)
       (effects (font (size 1.27 1.27)) hide)
     )
@@
     (property "Reference" "R11" (id 0) (at 52.07 38.1 90))
     (property "Value" "150R" (id 1) (at 52.07 39.37 90))
-    (property "Footprint" "" (id 2) (at 52.07 41.148 90)
+    (property "Footprint" "Resistor_SMD:R_0603_1608Metric" (id 2) (at 52.07 41.148 90)
       (effects (font (size 1.27 1.27)) hide)
     )
@@
     (property "Reference" "R18" (id 0) (at 95.25 38.1 90))
     (property "Value" "150R" (id 1) (at 95.25 39.37 90))
-    (property "Footprint" "" (id 2) (at 95.25 41.148 90)
+    (property "Footprint" "Resistor_SMD:R_0603_1608Metric" (id 2) (at 95.25 41.148 90)
       (effects (font (size 1.27 1.27)) hide)
     )
@@
     (property "Reference" "R31" (id 0) (at 95.25 50.8 90))
     (property "Value" "150R" (id 1) (at 95.25 52.07 90))
-    (property "Footprint" "" (id 2) (at 95.25 53.848 90)
+    (property "Footprint" "Resistor_SMD:R_0603_1608Metric" (id 2) (at 95.25 53.848 90)
       (effects (font (size 1.27 1.27)) hide)
     )
@@
       (effects (font (size 1.27 1.27)) (justify left))
     )
-    (property "Footprint" "" (id 2) (at 26.162 36.83 90)
+    (property "Footprint" "Resistor_SMD:R_0402_1005Metric" (id 2) (at 26.162 36.83 90)
       (effects (font (size 1.27 1.27)) hide)
     )
@@
     (property "Reference" "R12" (id 0) (at 52.07 40.64 90))
     (property "Value" "150R" (id 1) (at 52.07 41.91 90))
-    (property "Footprint" "" (id 2) (at 52.07 43.688 90)
+    (property "Footprint" "Resistor_SMD:R_0603_1608Metric" (id 2) (at 52.07 43.688 90)
       (effects (font (size 1.27 1.27)) hide)
     )
@@
     (property "Reference" "R17" (id 0) (at 95.25 35.56 90))
     (property "Value" "150R" (id 1) (at 95.25 36.83 90))
-    (property "Footprint" "" (id 2) (at 95.25 38.608 90)
+    (property "Footprint" "Resistor_SMD:R_0603_1608Metric" (id 2) (at 95.25 38.608 90)
       (effects (font (size 1.27 1.27)) hide)
     )
@@
     (property "Reference" "R14" (id 0) (at 52.07 45.72 90))
     (property "Value" "150R" (id 1) (at 52.07 46.99 90))
-    (property "Footprint" "" (id 2) (at 52.07 48.768 90)
+    (property "Footprint" "Resistor_SMD:R_0603_1608Metric" (id 2) (at 52.07 48.768 90)
       (effects (font (size 1.27 1.27)) hide)
     )
@@
     (property "Reference" "R20" (id 0) (at 95.25 43.18 90))
     (property "Value" "150R" (id 1) (at 95.25 44.45 90))
-    (property "Footprint" "" (id 2) (at 95.25 46.228 90)
+    (property "Footprint" "Resistor_SMD:R_0603_1608Metric" (id 2) (at 95.25 46.228 90)
       (effects (font (size 1.27 1.27)) hide)
     )
@@
     (property "Reference" "R15" (id 0) (at 52.07 48.26 90))
     (property "Value" "150R" (id 1) (at 52.07 49.53 90))
-    (property "Footprint" "" (id 2) (at 52.07 51.308 90)
+    (property "Footprint" "Resistor_SMD:R_0603_1608Metric" (id 2) (at 52.07 51.308 90)
       (effects (font (size 1.27 1.27)) hide)
     )
@@
   (symbol (lib_id "power:GND") (at 137.16 56.515 0) (unit 1)
     (in_bom yes) (on_board yes) (fields_autoplaced)
-    (property "Reference" "#PWR071" (id 0) (at 137.16 62.865 0)
+    (property "Reference" "#PWR0129" (id 0) (at 137.16 62.865 0)
       (effects (font (size 1.27 1.27)) hide)
     )
@@
   (symbol (lib_id "power:GND") (at 130.175 56.515 0) (unit 1)
     (in_bom yes) (on_board yes) (fields_autoplaced)
-    (property "Reference" "#PWR011" (id 0) (at 130.175 62.865 0)
+    (property "Reference" "#PWR0130" (id 0) (at 130.175 62.865 0)
       (effects (font (size 1.27 1.27)) hide)
     )
@@
     (property "Reference" "R30" (id 0) (at 95.25 48.26 90))
     (property "Value" "150R" (id 1) (at 95.25 49.53 90))
-    (property "Footprint" "" (id 2) (at 95.25 51.308 90)
-      (effects (font (size 1.27 1.27)) hide)
-    )
+    (property "Footprint" "Resistor_SMD:R_0603_1608Metric" (id 2) (at 95.25 51.308 90)
+      (effects (font (size 1.27 1.27)) hide)
+    )
